Commit message: ros2 compat

File: dsr_description/urdf/e0509.urdf (robot description, URDF)
Before this commit: robot e0509, 8 links, 7 joints
Links:
- removed link base_0
- removed link link1
- removed link link2
- removed link link3
- removed link link4
- removed link link5
- removed link link6
- added link base_link, mass 1.803; visual mesh filename=package://dsr_description/meshes/e0509/E0509_0_0.dae scale=0.001 0.001 0.001
- added link link_1, mass 5.75; visual mesh filename=package://dsr_description/meshes/e0509/E0509_1_1.dae scale=0.001 0.001 0.001; visual mesh filename=package://dsr_description/meshes/e0509/E0509_1_2.dae scale=0.001 0.001 0.001
- added link link_2, mass 3.461; visual mesh filename=package://dsr_description/meshes/e0509/E0509_2_1.dae scale=0.001 0.001 0.001; visual mesh filename=package://dsr_description/meshes/e0509/E0509_2_2.dae scale=0.001 0.001 0.001
- added link link_3, mass 4.582; visual mesh filename=package://dsr_description/meshes/e0509/E0509_3_1.dae scale=0.001 0.001 0.001; visual mesh filename=package://dsr_description/meshes/e0509/E0509_3_2.dae scale=0.001 0.001 0.001
- added link link_4, mass 2.207; visual mesh filename=package://dsr_description/meshes/e0509/E0509_4_1.dae scale=0.001 0.001 0.001; visual mesh filename=package://dsr_description/meshes/e0509/E0509_4_2.dae scale=0.001 0.001 0.001
- added link link_5, mass 3.545; visual mesh filename=package://dsr_description/meshes/e0509/E0509_5_1.dae scale=0.001 0.001 0.001; visual mesh filename=package://dsr_description/meshes/e0509/E0509_5_2.dae scale=0.001 0.001 0.001
- added link link_6, mass 0.721; visual mesh filename=package://dsr_description/meshes/e0509/E0509_6_1.dae scale=0.001 0.001 0.001
Joints:
- removed joint joint1
- removed joint joint2
- removed joint joint3
- removed joint joint4
- removed joint joint5
- removed joint joint6
- added joint joint_1: type revolute, parent base_link, child link_1, origin xyz=0 0 0.2045 rpy=0 0 0, axis 0 0 1, limit lower=-6.2832 upper=6.2832 effort=194 velocity=3.1416
- added joint joint_2: type revolute, parent link1, child link_2, origin xyz=0  0  0 rpy=0     -1.5708     -1.5708, axis 0 0 1, limit lower=-6.2832 upper=6.2832 effort=194 velocity=3.1416
- added joint joint_3: type revolute, parent link2, child link_3, origin xyz=0.373           0           0 rpy=0           0      1.5708, axis 0 0 1, limit lower=-2.7053 upper=2.7053 effort=194 velocity=3.1416
- added joint joint_4: type revolute, parent link3, child link_4, origin xyz=0      -0.373           0 rpy=1.5708           0           0, axis 0 0 1, limit lower=-6.2832 upper=6.2832 effort=66 velocity=3.927
- added joint joint_5: type revolute, parent link4, child link_5, origin xyz=0  0  0 rpy=-1.5708           0           0, axis 0 0 1, limit lower=-6.2832 upper=6.2832 effort=66 velocity=3.927
- added joint joint_6: type revolute, parent link5, child link_6, origin xyz=0     -0.1725           0 rpy=1.5708           0           0, axis 0 0 1, limit lower=-6.2832 upper=6.2832 effort=66 velocity=3.927
- joint fixed: child base_0 -> base_link

File: dsr_description/xacro/macro.a0509.white.xacro (robot description, xacro)
@@ -6,5 +6,5 @@
 	<xacro:macro name="a0509" params="namespace">
 		<xacro:dsr_materials />
-		<link name="base_0">
+		<link name="base_link">
 			<inertial>
 				<mass value="2.198"/>
@@ -29,5 +29,5 @@
 		<!-- joint 1 -->
 		<joint name="joint1" type="revolute">
-			<parent link="base_0" />
+			<parent link="base_link" />
 			<child link="link1" />
 			<origin rpy="0 0 0" xyz="0 0 0.1555" />

File: dsr_description/xacro/macro.e0509.white.xacro (robot description, xacro)
@@ -6,5 +6,5 @@
 	<xacro:macro name="e0509" params="namespace">
 		<xacro:dsr_materials />
-		<link name="base_0">
+		<link name="base_link">
 			<inertial>
         <mass value="1.803"/>
@@ -26,7 +26,7 @@
 		</link>
 		<!-- joint 1 -->
-		<joint name="joint1" type="revolute">
-			<parent link="base_0" />
-			<child link="link1" />
+		<joint name="joint_1" type="revolute">
+			<parent link="base_link" />
+			<child link="link_1" />
 			<origin rpy="0 0 0" xyz="0 0 0.2045"/>
       <axis xyz="0 0 1"/>
@@ -34,5 +34,5 @@
 			<dynamics friction="0" />
 		</joint>
-		<link name="link1">
+		<link name="link_1">
 			<inertial>
         <mass value="5.75"/>
@@ -90,7 +90,7 @@
 		</link>
 		<!-- joint2 -->
-		<joint name="joint2" type="revolute">
-			<parent link="link1" />
-			<child link="link2" />
+		<joint name="joint_2" type="revolute">
+			<parent link="link_1" />
+			<child link="link_2" />
 			<origin rpy="0 -1.5708 -1.5708" xyz="0 0 0"/>
       <axis xyz="0 0 1"/>
@@ -98,5 +98,5 @@
 			<dynamics friction="0" />
 		</joint>
-		<link name="link2">
+		<link name="link_2">
 			<inertial>
 				<mass value="3.461"/>
@@ -130,7 +130,7 @@
 		</link>
 		<!-- joint3 -->
-		<joint name="joint3" type="revolute">
-			<parent link="link2" />
-			<child link="link3" />
+		<joint name="joint_3" type="revolute">
+			<parent link="link_2" />
+			<child link="link_3" />
 			<origin rpy="0 0 1.5708" xyz="0.373 0 0"/>
       <axis xyz="0 0 1"/>
@@ -138,5 +138,5 @@
 			<dynamics friction="0" />
 		</joint>
-		<link name="link3">
+		<link name="link_3">
 			<inertial>
 				<mass value="4.582"/>
@@ -170,7 +170,7 @@
 		</link>
 		<!-- joint4 -->
-		<joint name="joint4" type="revolute">
-			<parent link="link3" />
-			<child link="link4" />
+		<joint name="joint_4" type="revolute">
+			<parent link="link_3" />
+			<child link="link_4" />
 			<origin rpy="1.5708 0 0" xyz="0 -0.373 0"/>
       <axis xyz="0 0 1"/>
@@ -178,5 +178,5 @@
 			<dynamics friction="0" />
 		</joint>
-		<link name="link4">
+		<link name="link_4">
 			<inertial>
 				<mass value="2.207"/>
@@ -210,7 +210,7 @@
 		</link>
 		<!-- joint5 -->
-		<joint name="joint5" type="revolute">
-			<parent link="link4" />
-			<child link="link5" />
+		<joint name="joint_5" type="revolute">
+			<parent link="link_4" />
+			<child link="link_5" />
 			<origin rpy="-1.5708 0 0" xyz="0 0 0"/>
       <axis xyz="0 0 1"/>
@@ -218,5 +218,5 @@
 			<dynamics friction="0" />
 		</joint>
-		<link name="link5">
+		<link name="link_5">
 			<inertial>
 				<mass value="3.545"/>
@@ -250,7 +250,7 @@
 		</link>
 		<!-- joint6 -->
-		<joint name="joint6" type="revolute">
-			<parent link="link5" />
-			<child link="link6" />
+		<joint name="joint_6" type="revolute">
+			<parent link="link_5" />
+			<child link="link_6" />
 			<origin rpy="1.5708 0 0" xyz="0 -0.1725 0"/>
       <axis xyz="0 0 1"/>
@@ -258,5 +258,5 @@
 			<dynamics friction="0" />
 		</joint>
-		<link name="link6">
+		<link name="link_6">
 			<inertial>
 				<mass value="0.721"/>
